File: Eagle Files/ESP8266_BREAKOUT.brd (EAGLE design)
At the start: 43.2 x 30.5 mm, 17 parts, among them U2 LM1117-3V3-T0-220

Commit message: Update Eagle Files
Parts:
- removed J5: (no value), con-lstb:MA04-1
- J4: value (none) -> HEADER-ESP8266-4X2; device con-lstb:MA04-1 -> HEADER-4X2-A:HEADER-4X2-A
- moved J4 3.30 mm to (38.1, 18.5), turned to 270 degrees
Connections:
- net !RST: now also J4.3; no longer J4.2, S1.3
- net +3V3: now also J4.4; no longer J4.1
- net CH_PD: now also J4.2; no longer J4.3
- net GND: now also J4.5; no longer J5.4, S1.1, S2.1
- net GPIO0: now also J4.7; no longer J5.2, S2.3
- net GPIO2: now also J4.6; no longer J5.3
- net RX_PC: now also J4.1; no longer J4.4
- net TX: now also J4.8; no longer J5.1
Routing:
- net GND: track 6.50 -> 0.00 mm
- net !RST: track 25.9 -> 26.5 mm
- net CH_PD: track 22.2 -> 22.7 mm
- net RX_PC: track 36.0 -> 36.5 mm
