File: Eagle Files/ESP8266_BREAKOUT.sch (EAGLE design)
At the start: 17 parts, among them U2 LM1117-3V3-T0-220

Commit message: Update Eagle Files
Parts:
- removed J5: (no value), con-lstb:MA04-1
- J4: value (none) -> HEADER-ESP8266-4X2; device con-lstb:MA04-1 -> HEADER-4X2-A:HEADER-ESP8266-4X2
Connections:
- net !RST: now also J4.3; no longer J4.2, S1.3
- net +3V3: now also J4.4; no longer J4.1
- net CH_PD: now also J4.2; no longer J4.3
- net GND: now also J4.5; no longer J5.4, S1.1, S2.1
- net GPIO0: now also J4.7; no longer J5.2, S2.3
- net GPIO2: now also J4.6; no longer J5.3
- net RX_PC: now also J4.1; no longer J4.4
- net TX: now also J4.8; no longer J5.1
Other:
- moved on the sheet: S1, S2
Changed lines of the file:
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@@
 <part name="SUPPLY6" library="supply2" deviceset="GND" device=""/>
 <part name="J3" library="con-lstb" deviceset="MA03-1" device=""/>
-<part name="J4" library="con-lstb" deviceset="MA04-1" device=""/>
-<part name="J5" library="con-lstb" deviceset="MA04-1" device=""/>
 <part name="+3V3" library="supply1" deviceset="+3V3" device=""/>
 <part name="+3V4" library="supply1" deviceset="+3V3" device=""/>
@@
 <part name="S2" library="1825910-6" deviceset="1825910-6-SPST-NOPB-4P" device=""/>
 <part name="FRAME1" library="frames" deviceset="LETTER_L" device=""/>
+<part name="J4" library="HEADER-4X2-A" deviceset="HEADER-ESP8266-4X2" device=""/>
 </parts>
 <sheets>
 <sheet>
 <plain>
-<text x="205.74" y="111.76" size="1.778" layer="91">TX from ESP8266</text>
-<text x="205.74" y="81.28" size="1.778" layer="91">RX to ESP8266</text>
+<text x="170.18" y="109.22" size="1.778" layer="91">TX from ESP8266</text>
+<text x="170.18" y="73.66" size="1.778" layer="91">RX to ESP8266</text>
 </plain>
 <instances>
@@
 <instance part="SUPPLY6" gate="GND" x="88.9" y="86.36"/>
 <instance part="J3" gate="G$1" x="129.54" y="104.14" rot="MR0"/>
-<instance part="J4" gate="1" x="203.2" y="114.3" rot="R180"/>
-<instance part="J5" gate="1" x="203.2" y="76.2" rot="R180"/>
 <instance part="+3V3" gate="G$1" x="190.5" y="139.7"/>
 <instance part="+3V4" gate="G$1" x="160.02" y="139.7"/>
 <instance part="+3V5" gate="G$1" x="167.64" y="139.7"/>
-<instance part="SUPPLY7" gate="GND" x="190.5" y="66.04"/>
+<instance part="SUPPLY7" gate="GND" x="228.6" y="71.12"/>
 <instance part="+3V6" gate="G$1" x="160.02" y="104.14"/>
 <instance part="SUPPLY8" gate="GND" x="119.38" y="78.74" rot="R270"/>
@@
 <attribute name="VALUE" x="73.66" y="152.4" size="1.778" layer="96" display="off"/>
 </instance>
-<instance part="S1" gate="G$1" x="127" y="116.84" smashed="yes">
-<attribute name="NAME" x="132.08" y="121.158" size="1.778" layer="95"/>
-<attribute name="VALUE" x="132.08" y="110.998" size="1.778" layer="96" display="off"/>
-</instance>
-<instance part="S2" gate="G$1" x="127" y="78.74" smashed="yes">
-<attribute name="NAME" x="132.08" y="83.058" size="1.778" layer="95"/>
-<attribute name="VALUE" x="132.08" y="72.898" size="1.778" layer="96" display="off"/>
+<instance part="S1" gate="G$1" x="127" y="119.38" smashed="yes">
+<attribute name="NAME" x="132.08" y="123.698" size="1.778" layer="95"/>
+<attribute name="VALUE" x="132.08" y="113.538" size="1.778" layer="96" display="off"/>
+</instance>
+<instance part="S2" gate="G$1" x="127" y="81.28" smashed="yes">
+<attribute name="NAME" x="132.08" y="85.598" size="1.778" layer="95"/>
+<attribute name="VALUE" x="132.08" y="75.438" size="1.778" layer="96" display="off"/>
 </instance>
 <instance part="FRAME1" gate="G$1" x="0" y="0"/>
 <instance part="FRAME1" gate="G$2" x="147.32" y="0"/>
+<instance part="J4" gate="G$1" x="195.58" y="119.38"/>
 </instances>
 <busses>
@@
 </segment>
 <segment>
-<pinref part="J5" gate="1" pin="4"/>
-<wire x1="195.58" y1="73.66" x2="190.5" y2="73.66" width="0.1524" layer="91"/>
 <pinref part="SUPPLY7" gate="GND" pin="GND"/>
-<wire x1="190.5" y1="73.66" x2="190.5" y2="68.58" width="0.1524" layer="91"/>
+<wire x1="228.6" y1="73.66" x2="228.6" y2="111.76" width="0.1524" layer="91"/>
+<pinref part="J4" gate="G$1" pin="5"/>
+<wire x1="228.6" y1="111.76" x2="220.98" y2="111.76" width="0.1524" layer="91"/>
 </segment>
 <segment>
@@
 </segment>
 <segment>
-<pinref part="SUPPLY9" gate="GND" pin="GND"/>
-<wire x1="127" y1="116.84" x2="121.92" y2="116.84" width="0.1524" layer="91"/>
-<wire x1="127" y1="116.84" x2="127" y2="114.3" width="0.1524" layer="91"/>
-<pinref part="S1" gate="G$1" pin="1"/>
-<junction x="127" y="116.84"/>
-<pinref part="S1" gate="G$1" pin="2"/>
-</segment>
-<segment>
-<pinref part="SUPPLY8" gate="GND" pin="GND"/>
-<wire x1="121.92" y1="78.74" x2="127" y2="78.74" width="0.1524" layer="91"/>
-<wire x1="127" y1="78.74" x2="127" y2="76.2" width="0.1524" layer="91"/>
-<pinref part="S2" gate="G$1" pin="1"/>
-<junction x="127" y="78.74"/>
-<pinref part="S2" gate="G$1" pin="2"/>
-</segment>
-<segment>
 <pinref part="SUPPLY3" gate="GND" pin="GND"/>
 <pinref part="U2" gate="G$1" pin="GND"/>
 <wire x1="71.12" y1="149.86" x2="71.12" y2="152.4" width="0.1524" layer="91"/>
+</segment>
+<segment>
+<pinref part="SUPPLY8" gate="GND" pin="GND"/>
+<pinref part="S2" gate="G$1" pin="2"/>
+<wire x1="121.92" y1="78.74" x2="127" y2="78.74" width="0.1524" layer="91"/>
+</segment>
+<segment>
+<pinref part="SUPPLY9" gate="GND" pin="GND"/>
+<pinref part="S1" gate="G$1" pin="2"/>
+<wire x1="121.92" y1="116.84" x2="127" y2="116.84" width="0.1524" layer="91"/>
 </segment>
 </net>
@@
 </segment>
 <segment>
-<pinref part="J4" gate="1" pin="1"/>
 <wire x1="195.58" y1="119.38" x2="190.5" y2="119.38" width="0.1524" layer="91"/>
 <pinref part="+3V3" gate="G$1" pin="+3V3"/>
 <wire x1="190.5" y1="119.38" x2="190.5" y2="137.16" width="0.1524" layer="91"/>
+<pinref part="J4" gate="G$1" pin="4"/>
 </segment>
 <segment>
@@
 </segment>
 <segment>
-<pinref part="J4" gate="1" pin="4"/>
 <wire x1="195.58" y1="111.76" x2="152.4" y2="111.76" width="0.1524" layer="91"/>
 <label x="172.72" y="111.76" size="1.778" layer="95"/>
+<pinref part="J4" gate="G$1" pin="1"/>
 </segment>
 </net>
@@
 </segment>
 <segment>
-<pinref part="J5" gate="1" pin="1"/>
-<wire x1="195.58" y1="81.28" x2="152.4" y2="81.28" width="0.1524" layer="91"/>
+<wire x1="236.22" y1="81.28" x2="152.4" y2="81.28" width="0.1524" layer="91"/>
 <label x="172.72" y="81.28" size="1.778" layer="95" font="vector"/>
+<wire x1="236.22" y1="81.28" x2="236.22" y2="119.38" width="0.1524" layer="91"/>
+<pinref part="J4" gate="G$1" pin="8"/>
+<wire x1="236.22" y1="119.38" x2="220.98" y2="119.38" width="0.1524" layer="91"/>
 </segment>
 </net>
 <net name="!RST" class="0">
 <segment>
-<pinref part="J4" gate="1" pin="2"/>
 <wire x1="195.58" y1="116.84" x2="167.64" y2="116.84" width="0.1524" layer="91"/>
 <label x="172.72" y="116.84" size="1.778" layer="95"/>
-<wire x1="167.64" y1="116.84" x2="144.78" y2="116.84" width="0.1524" layer="91"/>
 <pinref part="R2" gate="G$1" pin="2"/>
 <wire x1="167.64" y1="116.84" x2="167.64" y2="121.92" width="0.1524" layer="91"/>
+<pinref part="J4" gate="G$1" pin="3"/>
+<pinref part="S1" gate="G$1" pin="4"/>
+<wire x1="144.78" y1="116.84" x2="167.64" y2="116.84" width="0.1524" layer="91"/>
 <junction x="167.64" y="116.84"/>
-<wire x1="144.78" y1="116.84" x2="144.78" y2="114.3" width="0.1524" layer="91"/>
-<pinref part="S1" gate="G$1" pin="3"/>
-<junction x="144.78" y="116.84"/>
-<pinref part="S1" gate="G$1" pin="4"/>
 </segment>
 </net>
 <net name="CH_PD" class="0">
 <segment>
-<pinref part="J4" gate="1" pin="3"/>
 <wire x1="195.58" y1="114.3" x2="160.02" y2="114.3" width="0.1524" layer="91"/>
 <label x="172.72" y="114.3" size="1.778" layer="95"/>
@@
 <wire x1="160.02" y1="121.92" x2="160.02" y2="114.3" width="0.1524" layer="91"/>
 <junction x="160.02" y="114.3"/>
+<pinref part="J4" gate="G$1" pin="2"/>
 </segment>
 </net>
@@
 </segment>
 <segment>
-<pinref part="J5" gate="1" pin="2"/>
-<wire x1="195.58" y1="78.74" x2="144.78" y2="78.74" width="0.1524" layer="91"/>
+<wire x1="233.68" y1="78.74" x2="144.78" y2="78.74" width="0.1524" layer="91"/>
 <label x="172.72" y="78.74" size="1.778" layer="95" font="vector"/>
-<wire x1="144.78" y1="78.74" x2="144.78" y2="76.2" width="0.1524" layer="91"/>
-<pinref part="S2" gate="G$1" pin="3"/>
-<junction x="144.78" y="78.74"/>
+<wire x1="233.68" y1="78.74" x2="233.68" y2="116.84" width="0.1524" layer="91"/>
+<pinref part="J4" gate="G$1" pin="7"/>
+<wire x1="233.68" y1="116.84" x2="220.98" y2="116.84" width="0.1524" layer="91"/>
 <pinref part="S2" gate="G$1" pin="4"/>
 </segment>
@@
 <net name="GPIO2" class="0">
 <segment>
-<pinref part="J5" gate="1" pin="3"/>
-<wire x1="195.58" y1="76.2" x2="160.02" y2="76.2" width="0.1524" layer="91"/>
 <label x="172.72" y="76.2" size="1.778" layer="95" font="vector"/>
 <pinref part="R3" gate="G$1" pin="2"/>
@@
 <wire x1="160.02" y1="76.2" x2="160.02" y2="86.36" width="0.1524" layer="91"/>
 <junction x="160.02" y="76.2"/>
+<wire x1="160.02" y1="76.2" x2="231.14" y2="76.2" width="0.1524" layer="91"/>
+<wire x1="231.14" y1="76.2" x2="231.14" y2="114.3" width="0.1524" layer="91"/>
+<pinref part="J4" gate="G$1" pin="6"/>
+<wire x1="231.14" y1="114.3" x2="220.98" y2="114.3" width="0.1524" layer="91"/>
 </segment>
 </net>
@@
 </sheet>
 </sheets>
-<errors>
-</errors>
 </schematic>
 </drawing>
